File: cad/electronics/lsm/lsm.sch (KiCad schematic (older format))
At the start: 18 parts, among them J1 Conn_01x02_Female, J2 Conn_01x02_Female, P1 Digital, P2 Analog, P3 CONN_01X01, P4 CONN_01X01, P5 CONN_01X01, P6 CONN_01X01, T1 2N2222, T2 2N2222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

Commit message: Almost finished with schematic.
Parts:
- removed P3, P4, P5, P6: CONN_01X01, Socket_Arduino_Nano:1pin_Nano, symbol Connector_Generic:Conn_01x01
- added C1, C3: 0.1uF, symbol Device:C
- added C2, C4: 47pF, symbol Device:C
- added D1, D2, D3, D?: LED, symbol Device:LED
- added J3: 6-8Ω coil, symbol Connector:Conn_01x02_Female
- added J4: Laser Diode, symbol Connector:Conn_01x02_Female
- added J5, J6: Conn_01x07_Female, symbol Connector:Conn_01x07_Female
- added M?: Fan, symbol Motor:Fan
- added Q3, Q4: TIP31C, pth-semi:TO-220, symbol semi-trans-generic:TIP31C
- added R10, R9: 4.7K, symbol Device:R_US
- added R3, R5, R6, R7, R8, R?: 1K, symbol Device:R_US
- added R4: 15, symbol Device:R_US
- added RV3: 1K, symbol Device:R_POT_US
- added RV4, RV5: 500K, symbol Device:R_POT_US
- added U4: LM317_TO-220, Package_TO_SOT_THT:TO-220-3_Vertical, symbol Regulator_Linear:LM317_TO-220
- J1, J2: value Conn_01x02_Female -> 8Ω speaker
- Q1: renamed from T1; symbol adafruit:2N2222 -> lsm-rescue:2N2222-adafruit
- Q2: renamed from T2; symbol adafruit:2N2222 -> lsm-rescue:2N2222-adafruit
Connections:
- net +3V3: now also R6.2
- net +5V: now also C1.2, C3.2, J3.1 (Pin_1), J5.2 (Pin_2), J5.6 (Pin_6), J5.7 (Pin_7), J6.2 (Pin_2), J6.6 (Pin_6), J6.7 (Pin_7), U4.3 (VI)
- net 0(Rx): now also B1.HV4 (HV_TXO_2); no longer B1.HV2 (HV_RXI_1)
- net 1(Tx): now also B1.HV3 (HV_RXI_2); no longer B1.HV1 (HV_TXO_1)
- net 3vRx: now also B1.LV3 (LV_RXO_2); no longer B1.LV1 (LV_TXI_1)
- net 3vTx: now also B1.LV4 (LV_TXI_2); no longer B1.LV2 (LV_RXO_1)
- net A0: now also C2.1, J5.4 (Pin_4), J5.5 (Pin_5), R9.2
- net A1: now also C4.1, J6.4 (Pin_4), J6.5 (Pin_5), R10.2
- net A2: now also J4.1 (Pin_1), R4.1, RV3.3, U4.1 (ADJ)
- net GND: now also B1.GND1 (GND), C1.1, C3.1, D1.1 (K), D2.1 (K), D3.1 (K), D?.1 (K), J5.3 (Pin_3), J6.3 (Pin_3), Q3.3 (E), Q4.3 (E); no longer B1.GND2 (GND)
- net SCL: now also B1.LV1 (LV_TXI_1); no longer B1.LV3 (LV_RXO_2)
- net SDA: now also B1.LV2 (LV_RXO_1); no longer B1.LV4 (LV_TXI_2)
- net IO15: now reaches U1.22 (15)
- net IO15: now also R3.2
- net IO13: now reaches U1.23 (13)
- net IO13: now also R7.2
- net IO12: now reaches U1.24 (12)
- net IO12: now also R5.2, R8.2
- net IO14: now reaches U1.25 (14)
- net IO14: now also R?.2
- net at U2.5 (SCL), U3.5 (SCL): now also B1.HV1 (HV_TXO_1); no longer B1.HV3 (HV_RXI_2)
- net at U2.4 (SDA), U3.4 (SDA): now also B1.HV2 (HV_RXI_1); no longer B1.HV4 (HV_TXO_2)
- new net: R4.2, RV3.1, RV3.2, U4.2 (VO)
- new net: Q3.1 (B), R5.1
- new net: J4.2 (Pin_2), Q3.2 (C)
- new net: D3.2 (A), R8.1
- new net: Q4.1 (B), R3.1
- new net: J3.2 (Pin_2), Q4.2 (C)
- new net: D2.2 (A), R7.1
- new net: D1.2 (A), R6.1
- new net: D?.2 (A), R?.1
- new net: C2.2, J5.1 (Pin_1), RV4.3
- new net: R9.1, RV4.1, RV4.2
- new net: C4.2, J6.1 (Pin_1), RV5.3
- new net: R10.1, RV5.1, RV5.2
- no-connect marks 14 -> 13
Other:
- note added: "Actuator drivers"
- note added: "Connected"
- note added: "Interface"
- note added: "Laser Driver"
- note added: "Laser on"
- note added: "Optical Sensor"
- note added: "Power"
- note added: "Request"
- note added: "Sensor Feedback"
- note added: "WCMCU-101 breakout board"
- note added: "X-axis\n"
- note added: "Y-axis"
- note added: "Z-axis"
- note removed: "Holes"
- moved on the sheet: B1, J1, J2, P1, P2, Q1, Q2, R1, R2, RV1, RV2, U1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
